File: pcb/poncho-max9924/poncho-max9924.sch (KiCad schematic (older format))
At the start: 48 parts, among them J1 Screw_Terminal_01x02, J2 Screw_Terminal_01x02, U1 MAX9924, U2 MAX9000

Commit message: Se agregaron modelos 3D de todos los componentes y sus footprints. Se re trabajo el posicionamiento de componentes en la placa.
Parts:
- removed JP5: jumper_4_open, misc:PinHeader_1x03_1x01_P2.54mm_Vertical, symbol custom_jumpers:jumper_4_open
- added J3: jumper_4_open, misc:PinHeader_1x03_1x01_P2.54mm_Vertical, symbol custom_jumpers:jumper_4_open
- U1: footprint umax:UMAX10 -> max9924:SOP50P490X110-10N; Manufacturer MAXIM -> (none)
- U2: footprint umax:UMAX8 -> max9000:SOP65P490X110-8N; Manufacturer MAXIM -> (none)
Changed lines of the file:
@@
 $EndDescr
-$Comp
-L Poncho_Esqueleto:Conn_Poncho2P_2x_20x2 XA1
-U 1 1 60EA4A8B
-P 2050 4650
-F 0 "XA1" H 2400 5100 60  0000 C CNN
-F 1 "Conn_Poncho2P_2x_20x2" H 2400 2900 60  0000 C CNN
-F 2 "Poncho_Esqueleto:Conn_Poncho_Mediano" H 2050 4650 60  0001 C CNN
-F 3 "" H 2050 4650 60  0000 C CNN
-	1    2050 4650
-	1    0    0    -1
-$EndComp
-$Comp
-L Poncho_Esqueleto:Conn_Poncho2P_2x_20x2 XA1
-U 2 1 60EA5F6F
-P 3850 4650
-F 0 "XA1" H 4200 5100 60  0000 C CNN
-F 1 "Conn_Poncho2P_2x_20x2" H 4200 2950 60  0000 C CNN
-F 2 "Poncho_Esqueleto:Conn_Poncho_Mediano" H 3850 4650 60  0001 C CNN
-F 3 "" H 3850 4650 60  0000 C CNN
-	2    3850 4650
-	1    0    0    -1
-$EndComp
 $Comp
 L Device:R_US R1
@@
 $EndComp
 $Comp
-L MAX9924-27:MAX9924 U1
-U 1 1 60F1B980
-P 4400 2450
-F 0 "U1" H 4400 3115 50  0000 C CNN
-F 1 "MAX9924" H 4400 3024 50  0000 C CNN
-F 2 "umax:UMAX10" H 4400 2450 50  0001 C CNN
-F 3 "https://www.maximintegrated.com/en/products/interface/sensor-interface/MAX9924.html/product-details/tabs-1" H 4400 2450 50  0001 C CNN
-F 4 "MAXIM" H 4400 2450 50  0001 C CNN "Manufacturer"
-	1    4400 2450
-	1    0    0    -1
-$EndComp
-$Comp
 L Jumper:Jumper_3_Open JP2
 U 1 1 60F22D1F
@@
 $EndComp
 $Comp
-L MAX9000:MAX9000 U2
-U 1 1 610BCF5D
-P 8900 2100
-F 0 "U2" H 8900 2565 50  0000 C CNN
-F 1 "MAX9000" H 8900 2474 50  0000 C CNN
-F 2 "umax:UMAX8" H 8950 2100 50  0001 C CNN
-F 3 "https://datasheets.maximintegrated.com/en/ds/MAX9000-MAX9005.pdf" H 8950 2100 50  0001 C CNN
-F 4 "MAXIM" H 8900 2100 50  0001 C CNN "Manufacturer"
-	1    8900 2100
-	1    0    0    -1
-$EndComp
-$Comp
 L power:GND #PWR012
 U 1 1 610CDC1D
@@
 F 3 "~" H 6200 3050 50  0001 C CNN
 	1    6200 3050
-	0    1    1    0
-$EndComp
-$Comp
-L custom_jumpers:jumper_4_open JP5
-U 1 1 610B4D80
-P 5550 2450
-F 0 "JP5" V 5400 2500 50  0000 L CNN
-F 1 "jumper_4_open" H 5600 2000 50  0001 C CNN
-F 2 "misc:PinHeader_1x03_1x01_P2.54mm_Vertical" H 5550 2450 50  0001 C CNN
-F 3 "" H 5550 2450 50  0001 C CNN
-	1    5550 2450
 	0    1    1    0
 $EndComp
@@
 	1    0    0    -1
 $EndComp
+$Comp
+L Poncho_Esqueleto:Conn_Poncho2P_2x_20x2 XA1
+U 1 1 6102D304
+P 2050 4650
+F 0 "XA1" H 2400 5197 60  0000 C CNN
+F 1 "Conn_Poncho2P_2x_20x2" H 2400 5091 60  0000 C CNN
+F 2 "Poncho_Esqueleto:Conn_Poncho_Mediano" H 2050 4650 60  0001 C CNN
+F 3 "" H 2050 4650 60  0000 C CNN
+	1    2050 4650
+	1    0    0    -1
+$EndComp
+$Comp
+L Poncho_Esqueleto:Conn_Poncho2P_2x_20x2 XA1
+U 2 1 610301F5
+P 3850 4650
+F 0 "XA1" H 4200 5197 60  0000 C CNN
+F 1 "Conn_Poncho2P_2x_20x2" H 4200 5091 60  0000 C CNN
+F 2 "Poncho_Esqueleto:Conn_Poncho_Mediano" H 3850 4650 60  0001 C CNN
+F 3 "" H 3850 4650 60  0000 C CNN
+	2    3850 4650
+	1    0    0    -1
+$EndComp
+$Comp
+L MAX9924-27:MAX9924 U1
+U 1 1 610364C6
+P 4400 2450
+F 0 "U1" H 4400 3115 50  0000 C CNN
+F 1 "MAX9924" H 4400 3024 50  0000 C CNN
+F 2 "max9924:SOP50P490X110-10N" H 4400 2450 50  0001 C CNN
+F 3 "" H 4400 2450 50  0001 C CNN
+	1    4400 2450
+	1    0    0    -1
+$EndComp
+$Comp
+L MAX9000:MAX9000 U2
+U 1 1 6103892E
+P 8900 2100
+F 0 "U2" H 8900 2565 50  0000 C CNN
+F 1 "MAX9000" H 8900 2474 50  0000 C CNN
+F 2 "max9000:SOP65P490X110-8N" H 8950 2100 50  0001 C CNN
+F 3 "" H 8950 2100 50  0001 C CNN
+	1    8900 2100
+	1    0    0    -1
+$EndComp
+$Comp
+L custom_jumpers:jumper_4_open J3
+U 1 1 6103959C
+P 5550 2450
+F 0 "J3" V 5600 2300 50  0000 L CNN
+F 1 "jumper_4_open" H 5600 2000 50  0001 C CNN
+F 2 "misc:PinHeader_1x03_1x01_P2.54mm_Vertical" H 5550 2445 50  0001 C CNN
+F 3 "" H 5550 2445 50  0001 C CNN
+	1    5550 2450
+	0    1    1    0
+$EndComp
 $EndSCHEMATC

Commit message: primer routeado
Other:
- note added: "NOTA 1: El pin 3 del integrado U1 esta etiquetado como "No Conectar"\n sin embargo en el esquemático está conectado a TP5 y R9. Esto está\n hecho así para respetar el diseño original del kit de evaluación que \nse está adaptando."
Changed lines of the file:
@@
 	0    1    1    0
 $EndComp
+Text Notes 8400 6500 0    50   ~ 0
+NOTA 1: El pin 3 del integrado U1 esta etiquetado como "No Conectar"\n sin embargo en el esquemático está conectado a TP5 y R9. Esto está\n hecho así para respetar el diseño original del kit de evaluación que \nse está adaptando.
 $EndSCHEMATC

Commit message: correcciones y ruteo listo, falta hacer U2 multiparte
Parts:
- added FID1, FID2, FID3, FID4: Fiducial, Fiducial:Fiducial_0.5mm_Mask1mm, symbol Mechanical:Fiducial
- added H1, H2: MountingHole, MountingHole:MountingHole_3.5mm_Pad, symbol Mechanical:MountingHole
- U1: Digikey PN (none) -> MAX9924UAUB+T
- U2: Digikey PN (none) -> MAX9000ESA+
- XA1: footprint Poncho_Esqueleto:Conn_Poncho_Mediano -> Poncho_Esqueleto:Conn_Poncho_SinBorde
Connections:
- wire segments 212 -> 215
Other:
- note added: "Agujeros de montaje y fiduciales"
Changed lines of the file:
@@
 encoding utf-8
 Sheet 1 1
-Title "Poncho MAX9924"
+Title "Poncho MAX9924: Interfaz para sensor de reluctancia variable"
 Date "2021-07-20"
 Rev "1"
@@
 $EndComp
 $Comp
-L power:GND #PWR07
-U 1 1 60F4090E
-P 3600 3400
-F 0 "#PWR07" H 3600 3150 50  0001 C CNN
-F 1 "GND" H 3605 3227 50  0001 C CNN
-F 2 "" H 3600 3400 50  0001 C CNN
-F 3 "" H 3600 3400 50  0001 C CNN
-	1    3600 3400
-	1    0    0    -1
-$EndComp
-$Comp
 L power:GND #PWR02
 U 1 1 60F485E5
@@
 	3850 3150 4250 3150
 Wire Wire Line
-	3600 3100 3600 3150
-Wire Wire Line
-	3850 3150 3600 3150
-Connection ~ 3850 3150
-Connection ~ 3600 3150
-Wire Wire Line
 	3400 2950 3450 2950
-Wire Wire Line
-	3450 2950 3450 3150
-Wire Wire Line
-	3450 3150 3600 3150
 Wire Wire Line
 	3150 2650 3150 2800
@@
 Wire Notes Line
 	11000 900  11000 3050
-Text Notes 9200 850  0    79   ~ 16
+Text Notes 7450 850  0    79   ~ 16
 Generador de onda triangular
 Wire Wire Line
@@
 Wire Wire Line
 	2700 1350 3000 1350
-$Comp
-L Connector:Screw_Terminal_01x02 J1
-U 1 1 61577878
-P 1200 1450
-F 0 "J1" H 1200 1200 50  0000 C CNN
-F 1 "Screw_Terminal_01x02" H 1118 1216 50  0001 C CNN
-F 2 "TerminalBlock:TerminalBlock_bornier-2_P5.08mm" H 1200 1450 50  0001 C CNN
-F 3 "~" H 1200 1450 50  0001 C CNN
-	1    1200 1450
-	-1   0    0    1
-$EndComp
 Wire Notes Line
 	750  900  7300 900
@@
 Wire Notes Line
 	750  3600 750  900
-Text Notes 6100 850  0    79   ~ 16
+Text Notes 750  850  0    79   ~ 16
 Contador de pulsos
 $Comp
@@
 	5500 2050 5550 2050
 Wire Wire Line
-	5550 2050 5550 1650
-Wire Wire Line
 	5550 1350 5400 1350
 Wire Wire Line
@@
 Wire Wire Line
 	4900 2250 5250 2250
-Connection ~ 5550 2050
 Wire Wire Line
 	5550 2250 5550 2050
@@
 Wire Notes Line
 	1700 3950 1700 6750
-Text Notes 4600 3950 0    79   ~ 16
+Text Notes 1700 3900 0    79   ~ 16
 Conectores EDU-CIAA
 Wire Wire Line
@@
 	2850 3300 2850 3400
 Wire Wire Line
-	3600 3150 3600 3400
-Wire Wire Line
 	1650 1350 1400 1350
 Wire Wire Line
@@
 F 0 "XA1" H 2400 5197 60  0000 C CNN
 F 1 "Conn_Poncho2P_2x_20x2" H 2400 5091 60  0000 C CNN
-F 2 "Poncho_Esqueleto:Conn_Poncho_Mediano" H 2050 4650 60  0001 C CNN
+F 2 "Poncho_Esqueleto:Conn_Poncho_SinBorde" H 2050 4650 60  0001 C CNN
 F 3 "" H 2050 4650 60  0000 C CNN
 	1    2050 4650
@@
 F 0 "XA1" H 4200 5197 60  0000 C CNN
 F 1 "Conn_Poncho2P_2x_20x2" H 4200 5091 60  0000 C CNN
-F 2 "Poncho_Esqueleto:Conn_Poncho_Mediano" H 3850 4650 60  0001 C CNN
+F 2 "Poncho_Esqueleto:Conn_Poncho_SinBorde" H 3850 4650 60  0001 C CNN
 F 3 "" H 3850 4650 60  0000 C CNN
 	2    3850 4650
@@
 F 1 "MAX9924" H 4400 3024 50  0000 C CNN
 F 2 "max9924:SOP50P490X110-10N" H 4400 2450 50  0001 C CNN
-F 3 "" H 4400 2450 50  0001 C CNN
+F 3 "https://datasheets.maximintegrated.com/en/ds/MAX9924-MAX9927.pdf" H 4400 2450 50  0001 C CNN
+F 4 "MAX9924UAUB+T" H 4400 2450 50  0001 C CNN "Digikey PN"
 	1    4400 2450
 	1    0    0    -1
@@
 F 1 "MAX9000" H 8900 2474 50  0000 C CNN
 F 2 "max9000:SOP65P490X110-8N" H 8950 2100 50  0001 C CNN
-F 3 "" H 8950 2100 50  0001 C CNN
+F 3 "https://datasheets.maximintegrated.com/en/ds/MAX9000-MAX9005.pdf" H 8950 2100 50  0001 C CNN
+F 4 "MAX9000ESA+" H 8900 2100 50  0001 C CNN "Digikey PN"
 	1    8900 2100
 	1    0    0    -1
@@
 Text Notes 8400 6500 0    50   ~ 0
 NOTA 1: El pin 3 del integrado U1 esta etiquetado como "No Conectar"\n sin embargo en el esquemático está conectado a TP5 y R9. Esto está\n hecho así para respetar el diseño original del kit de evaluación que \nse está adaptando.
+$Comp
+L Connector:Screw_Terminal_01x02 J1
+U 1 1 61577878
+P 1200 1350
+F 0 "J1" H 1200 1100 50  0000 C CNN
+F 1 "Screw_Terminal_01x02" H 1118 1116 50  0001 C CNN
+F 2 "TerminalBlock:TerminalBlock_bornier-2_P5.08mm" H 1200 1350 50  0001 C CNN
+F 3 "~" H 1200 1350 50  0001 C CNN
+	1    1200 1350
+	-1   0    0    -1
+$EndComp
+$Comp
+L power:GND #PWR0103
+U 1 1 611C1239
+P 5650 2100
+F 0 "#PWR0103" H 5650 1850 50  0001 C CNN
+F 1 "GND" H 5655 1927 50  0001 C CNN
+F 2 "" H 5650 2100 50  0001 C CNN
+F 3 "" H 5650 2100 50  0001 C CNN
+	1    5650 2100
+	1    0    0    -1
+$EndComp
+Wire Wire Line
+	5550 2050 5650 2050
+Wire Wire Line
+	5650 2050 5650 2100
+Connection ~ 5550 2050
+$Comp
+L power:GND #PWR0104
+U 1 1 611D3694
+P 3450 3200
+F 0 "#PWR0104" H 3450 2950 50  0001 C CNN
+F 1 "GND" H 3455 3027 50  0001 C CNN
+F 2 "" H 3450 3200 50  0001 C CNN
+F 3 "" H 3450 3200 50  0001 C CNN
+	1    3450 3200
+	1    0    0    -1
+$EndComp
+$Comp
+L power:GND #PWR0105
+U 1 1 611E15CE
+P 3850 3200
+F 0 "#PWR0105" H 3850 2950 50  0001 C CNN
+F 1 "GND" H 3855 3027 50  0001 C CNN
+F 2 "" H 3850 3200 50  0001 C CNN
+F 3 "" H 3850 3200 50  0001 C CNN
+	1    3850 3200
+	1    0    0    -1
+$EndComp
+Wire Wire Line
+	3850 3150 3850 3200
+Connection ~ 3850 3150
+Wire Wire Line
+	3450 2950 3450 3150
+Wire Wire Line
+	3450 3150 3600 3150
+Wire Wire Line
+	3600 3150 3600 3100
+Wire Wire Line
+	3450 3150 3450 3200
+Connection ~ 3450 3150
+$Comp
+L Mechanical:Fiducial FID1
+U 1 1 6123576E
+P 8450 4700
+F 0 "FID1" H 8535 4746 50  0000 L CNN
+F 1 "Fiducial" H 8535 4655 50  0000 L CNN
+F 2 "Fiducial:Fiducial_0.5mm_Mask1mm" H 8450 4700 50  0001 C CNN
+F 3 "~" H 8450 4700 50  0001 C CNN
+	1    8450 4700
+	1    0    0    -1
+$EndComp
+$Comp
+L Mechanical:Fiducial FID2
+U 1 1 612361A2
+P 8950 4700
+F 0 "FID2" H 9035 4746 50  0000 L CNN
+F 1 "Fiducial" H 9035 4655 50  0000 L CNN
+F 2 "Fiducial:Fiducial_0.5mm_Mask1mm" H 8950 4700 50  0001 C CNN
+F 3 "~" H 8950 4700 50  0001 C CNN
+	1    8950 4700
+	1    0    0    -1
+$EndComp
+$Comp
+L Mechanical:Fiducial FID3
+U 1 1 61236CC7
+P 8450 5150
+F 0 "FID3" H 8535 5196 50  0000 L CNN
+F 1 "Fiducial" H 8535 5105 50  0000 L CNN
+F 2 "Fiducial:Fiducial_0.5mm_Mask1mm" H 8450 5150 50  0001 C CNN
+F 3 "~" H 8450 5150 50  0001 C CNN
+	1    8450 5150
+	1    0    0    -1
+$EndComp
+$Comp
+L Mechanical:Fiducial FID4
+U 1 1 61284D9A
+P 8950 5150
+F 0 "FID4" H 9035 5196 50  0000 L CNN
+F 1 "Fiducial" H 9035 5105 50  0000 L CNN
+F 2 "Fiducial:Fiducial_0.5mm_Mask1mm" H 8950 5150 50  0001 C CNN
+F 3 "~" H 8950 5150 50  0001 C CNN
+	1    8950 5150
+	1    0    0    -1
+$EndComp
+$Comp
+L Mechanical:MountingHole H2
+U 1 1 612999F2
+P 7700 5150
+F 0 "H2" H 7800 5196 50  0000 L CNN
+F 1 "MountingHole" H 7800 5105 50  0000 L CNN
+F 2 "MountingHole:MountingHole_3.5mm_Pad" H 7700 5150 50  0001 C CNN
+F 3 "~" H 7700 5150 50  0001 C CNN
+	1    7700 5150
+	1    0    0    -1
+$EndComp
+$Comp
+L Mechanical:MountingHole H1
+U 1 1 6129A8A0
+P 7700 4700
+F 0 "H1" H 7800 4746 50  0000 L CNN
+F 1 "MountingHole" H 7800 4655 50  0000 L CNN
+F 2 "MountingHole:MountingHole_3.5mm_Pad" H 7700 4700 50  0001 C CNN
+F 3 "~" H 7700 4700 50  0001 C CNN
+	1    7700 4700
+	1    0    0    -1
+$EndComp
+Wire Notes Line
+	7500 4500 7500 5500
+Wire Notes Line
+	7500 5500 9500 5500
+Wire Notes Line
+	9500 5500 9500 4500
+Wire Notes Line
+	9500 4500 7500 4500
+Text Notes 7500 4450 0    79   ~ 16
+Agujeros de montaje y fiduciales
+$Comp
+L power:GND #PWR0106
+U 1 1 612F5A06
+P 7700 5250
+F 0 "#PWR0106" H 7700 5000 50  0001 C CNN
+F 1 "GND" H 7705 5077 50  0000 C CNN
+F 2 "" H 7700 5250 50  0001 C CNN
+F 3 "" H 7700 5250 50  0001 C CNN
+	1    7700 5250
+	1    0    0    -1
+$EndComp
+Wire Wire Line
+	7700 5150 7700 5250
+$Comp
+L power:GND #PWR0107
+U 1 1 613109F1
+P 7700 4800
+F 0 "#PWR0107" H 7700 4550 50  0001 C CNN
+F 1 "GND" H 7705 4627 50  0000 C CNN
+F 2 "" H 7700 4800 50  0001 C CNN
+F 3 "" H 7700 4800 50  0001 C CNN
+	1    7700 4800
+	1    0    0    -1
+$EndComp
+Wire Wire Line
+	7700 4700 7700 4800
 $EndSCHEMATC
